Commit message: AMAS support adjustments

File: urdf/vispa.urdf (robot description, URDF)
Before this commit: robot locarm, 10 links, 9 joints
Links:
- link link6: geometry collision mesh filename=package://vispa_description/meshes/LINK_5_col.stl scale=0.0001 0.0001 0.0001; visual mesh filename=package://vispa_description/meshes/LINK_5.stl scale=0.0001 0.0001 0.0001
Joints:
- joint j01: limit lower=-3.14149265359 upper=3.14149265359 effort=50 velocity=0.09395689 -> lower=-3.14149265359 upper=-0.174533 effort=50 velocity=0.09395689
- joint j23: axis 0 1 0 -> 0 -1 0; limit lower=-3.14149265359 upper=3.14149265359 effort=50 velocity=0.09395689 -> lower=-1.5707963268 upper=1.5707963268 effort=50 velocity=0.09395689
- joint j34: limit lower=-3.14149265359 upper=3.14149265359 effort=50 velocity=0.09395689 -> lower=0.174533 upper=3.14149265359 effort=50 velocity=0.09395689

File: urdf/vispa.xacro (robot description, xacro)
@@ -142,5 +142,5 @@
     <visual>
       <geometry>
-        <mesh filename="package://vispa_description/meshes/LINK_5.stl" scale="0.001 0.001 0.001"/>
+        <mesh filename="package://vispa_description/meshes/LINK_5.stl" scale="0.0001 0.0001 0.0001"/>
       </geometry>
     </visual>

Commit message: Update vispa.urdf

File: urdf/vispa.urdf (robot description, URDF)
Before this commit: robot locarm, 10 links, 9 joints
Joints:
- joint j01: limit lower=-3.14149265359 upper=-0.174533 effort=50 velocity=0.09395689 -> lower=-2.96706 upper=0 effort=50 velocity=0.09395689
- joint j34: limit lower=0.174533 upper=3.14149265359 effort=50 velocity=0.09395689 -> lower=-2.96706 upper=-0.174533 effort=50 velocity=0.09395689

Commit message: Updated the Joint 5 to avoid gripper collision

File: urdf/vispa.urdf (robot description, URDF)
Before this commit: robot locarm, 10 links, 9 joints
Joints:
- joint j45: limit lower=-3.14149265359 upper=3.14149265359 effort=50 velocity=0.09395689 -> lower=0.523599 upper=3.14149265359 effort=50 velocity=0.09395689
